File: DC_ESP32_Motor_Board_CAN.kicad_pcb (KiCad board)
At the start: 2 copper layers, 29.8 x 46.2 mm, 45 parts, among them IC1 VNH7100BASTR, IC2 TJA1050T_CM, IC3 LSM6DS3TR-C, J1 SM04B-SRSS-TB, J2 SM04B-SRSS-TB, J3 XT30PB, J4 XT30PB, J5 SM04B-SRSS-TB, J6 SM04B-SRSS-TB, J7 XT30PB, J8 Conn_01x03_Pin, Q1 BSS138, Q2 BSS138, SW1 DSHP04TJGER, U1 MOUDLE-SEEEDUINO-XIAO-ESP32C3

Commit message: Minor Trace Updates
Routing:
- net Net-(IC1-INB): track 8.01 -> 11.5 mm
- net Net-(IC1-INA): track 17.5 -> 20.0 mm
- net INA: track 5.44 -> 3.96 mm
- net DipV: track 37.9 -> 37.4 mm
- net RSENSE: vias 3 -> 5
- net GND: vias 19 -> 25
